File: electronics/KiCAD/Watch Winder.kicad_pcb (KiCad board)
At the start: 2 copper layers, 82 x 26 mm, 14 parts, among them J1 12V, J2 Sensor, J3 USB-C, J4 Motor, U1 L7805, U2 ESP32, U3 TMC2226

Commit message: PCB corrections
Other:
- board text added: "WWCROSS V1.3"
- board text removed: "WWCROSS V1.2"
Changed lines of the file:
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@@
 			(drillshape 0)
 			(scaleselection 1)
-			(outputdirectory "Out/V1.2/")
+			(outputdirectory "Out/V1.3/")
 		)
 	)
@@
 		(layer "Edge.Cuts")
 	)
-	(gr_text "WWCROSS V1.2"
+	(gr_text "WWCROSS V1.3"
 		(at 108.585 64.77 0)
 		(layer "F.Cu")
